Commit message: final commit of all files including readme

File: mmp30_description/urdf/mmp30.urdf.xacro (robot description, xacro)
@@ -7,5 +7,5 @@
    <xacro:include filename="$(find velodyne_description)/urdf/VLP-16.urdf.xacro"/>
   <VLP-16 parent="base_link" name="velodyne" topic="/velodyne_points" hz="10" samples="440" gpu="${gpu}">
-    <origin xyz="0 0 0.25" rpy="0 0 3.14159" />
+    <origin xyz=".1 0 .5" rpy="0 0 3.14159" />
   </VLP-16>
   <!-- <joint name="arm_rover_joint" type="fixed">
@@ -34,7 +34,7 @@
   <link name="base_link">
     <visual>
-      <origin xyz="${base_x_size * -.5} ${base_y_size * -.5} 0" rpy="0 0 0" />
+      <origin xyz="0 0 0" rpy="0 0 0" />
       <geometry>
-          <mesh filename="package://mmp30_description/meshes/MMP30.dae"/>
+          <mesh filename="package://MMp30-Main-assembly/meshes/FinalRobotURDF/Body.stl" scale="0.001 0.001 0.001"  />
       </geometry>
     </visual>
@@ -113,11 +113,6 @@
     <geometry>
       <mesh
-        filename="package://MMp30-Main-assembly/meshes/SensorBaseChassis.STL" />
-    </geometry>
-    <material
-      name="">
-      <color
-        rgba="0.79216 0.81961 0.93333 1" />
-    </material>
+        filename="package://MMp30-Main-assembly/meshes/FinalRobotURDF/Mainassembly.stl"  scale="0.001 0.001 0.001"  />
+    </geometry>
   </visual>
 </link>
@@ -126,6 +121,6 @@
   type="fixed">
   <origin
-    xyz="-.1 .80 -.175"
-    rpy="${(M_PI/180) * 10} ${(M_PI/180) * 153} ${(M_PI/180) * 53} " />
+    xyz="0 0 .05"
+    rpy="${(M_PI/180) * 0} ${(M_PI/180) * 0} ${(M_PI/180) * 0 } " />
   <parent
     link="base_link" />
@@ -137,4 +132,47 @@
     k_velocity="0" />
 </joint>
+  <gazebo reference="SensorBaseChassis">
+    <material>Gazebo/Grey</material>
+  </gazebo>
+<link
+  name="GPS">
+  <inertial>
+    <origin
+      rpy="0 0 0" />
+    <mass
+      value="1.7565" />
+    <inertia
+      ixx="0.046345"
+      ixy="-0.00014939"
+      ixz="1.1248E-08"
+      iyy="0.042797"
+      iyz="5.3201E-07"
+      izz="0.055575" />
+  </inertial>
+  <visual>
+    <origin
+      xyz="0 0 0"
+      rpy= "0 0 0"/>
+    <geometry>
+      <mesh
+        filename="package://MMp30-Main-assembly/meshes/FinalRobotURDF/GPS_Mount_Assembly_MMP30.stl"  scale="0.001 0.001 0.001"  />
+    </geometry>
+  </visual>
+</link>
+<joint
+  name="GPS_Joint"
+  type="fixed">
+  <origin
+    xyz="0 0 .1"
+    rpy="${(M_PI/180) * 0} ${(M_PI/180) * 0} ${(M_PI/180) * 0 } " />
+  <parent
+    link="base_link" />
+  <child
+    link="GPS" />
+  <axis
+    xyz="0 0 0" />
+  <safety_controller
+    k_velocity="0" />
+</joint>
 <!-- Nod Link -->
 <link name="nod_link">
@@ -148,5 +186,5 @@
     <origin xyz="0 0 0" rpy="0 0 0"/>
     <geometry>
-  <box size=".01 .01 .1"/>
+  <box size=".0001 .0001 .00001"/>
     </geometry>
     <material name="grey"/>
@@ -160,5 +198,5 @@
 <!-- Nod joint -->
 <joint name="nod_joint" type="continuous">
-  <origin xyz=".01 0 0" rpy="0 ${(M_PI/180) * 0} ${(M_PI/180) * 0}"/>
+  <origin xyz=".01 0 -.025" rpy="0 ${(M_PI/180) * 0} ${(M_PI/180) * 0}"/>
   <parent link="nod_link"/>
   <axis xyz="0 1 0" />
@@ -180,5 +218,5 @@
 <!-- Hokuyo joint -->
 <joint name="hokuyo_joint" type="prismatic">
-  <origin xyz=".05 0 1.2" rpy="${(M_PI/180) * 0} ${(M_PI/180) * 0} ${(M_PI/180) * 0}"/>
+  <origin xyz=".05 0 1.15" rpy="${(M_PI/180) * 0} ${(M_PI/180) * 0} ${(M_PI/180) * 0}"/>
   <parent link="base_link"/>
   <axis xyz="0 0 1" />
@@ -252,5 +290,5 @@
 <joint name="camera_joint" type="fixed">
   <axis xyz="0 1 0" />
-  <origin xyz="0 0 1.0" rpy="0 ${(M_PI/180) * 40} ${(M_PI/180) * 0}"/>
+  <origin xyz=".1 0 1.0" rpy="0 ${(M_PI/180) * 30} ${(M_PI/180) * 0}"/>
   <parent link="base_link"/>
   <child link="camera_link"/>
@@ -267,7 +305,6 @@
     <origin xyz="0 0 0" rpy="0 0 0"/>
     <geometry>
-  <box size="${camera_link} ${camera_link} ${camera_link}"/>
-    </geometry>
-    <material name="grey"/>
+      <mesh filename="package://mmp30_description/meshes/kinect.dae"/>
+    </geometry>
   </visual>
   <inertial>
@@ -277,7 +314,4 @@
   </inertial>
 </link>
-  <gazebo reference="camera_link">
-    <material>Gazebo/DarkGrey</material>
-  </gazebo>
 </xacro:macro>
 </robot>

File: mmp30_gazebo/urdf/mmp30.gazebo.xacro (robot description, xacro)
@@ -50,44 +50,40 @@
       </plugin>
     </gazebo>
-     <!-- camera -->
-  <gazebo reference="camera_link">
-    <sensor type="camera" name="camera1">
-      <update_rate>30.0</update_rate>
-      <camera name="head">
-        <horizontal_fov>1.3962634</horizontal_fov>
-        <image>
-          <width>800</width>
-          <height>800</height>
-          <format>R8G8B8</format>
-        </image>
-        <clip>
-          <near>0.02</near>
-          <far>300</far>
-        </clip>
-        <noise>
-          <type>gaussian</type>
-          <!-- Noise is sampled independently per pixel on each frame.
-               That pixel's noise value is added to each of its color
-               channels, which at that point lie in the range [0,1]. -->
-          <mean>0.0</mean>
-          <stddev>0.007</stddev>
-        </noise>
-      </camera>
-      <plugin name="camera_controller" filename="libgazebo_ros_camera.so">
-        <alwaysOn>true</alwaysOn>
-        <updateRate>0.0</updateRate>
-        <cameraName>mmp30/camera1</cameraName>
-        <imageTopicName>image_raw</imageTopicName>
-        <cameraInfoTopicName>camera_info</cameraInfoTopicName>
-        <frameName>camera_link</frameName>
-        <hackBaseline>0.07</hackBaseline>
-        <distortionK1>0.0</distortionK1>
-        <distortionK2>0.0</distortionK2>
-        <distortionK3>0.0</distortionK3>
-        <distortionT1>0.0</distortionT1>
-        <distortionT2>0.0</distortionT2>
-      </plugin>
-    </sensor>
-  </gazebo>
+<gazebo reference="camera_link">
+      <sensor type="depth" name="camera">
+        <always_on>true</always_on>
+        <update_rate>20.0</update_rate>
+        <camera>
+          <horizontal_fov>${60.0*M_PI/180.0}</horizontal_fov>
+          <image>
+            <format>B8G8R8</format>
+            <width>640</width>
+            <height>480</height>
+          </image>
+          <clip>
+            <near>0.05</near>
+            <far>8.0</far>
+          </clip>
+        </camera>
+        <plugin name="kinect_camera_controller" filename="libgazebo_ros_openni_kinect.so">
+          <cameraName>camera</cameraName>
+          <alwaysOn>true</alwaysOn>
+          <updateRate>10</updateRate>
+          <imageTopicName>rgb/image_raw</imageTopicName>
+          <depthImageTopicName>depth/image_raw</depthImageTopicName>
+          <pointCloudTopicName>depth/points</pointCloudTopicName>
+          <cameraInfoTopicName>rgb/camera_info</cameraInfoTopicName>
+          <depthImageCameraInfoTopicName>depth/camera_info</depthImageCameraInfoTopicName>
+          <frameName>camera_depth_optical_frame</frameName>
+          <baseline>0.1</baseline>
+          <distortion_k1>0.0</distortion_k1>
+          <distortion_k2>0.0</distortion_k2>
+          <distortion_k3>0.0</distortion_k3>
+          <distortion_t1>0.0</distortion_t1>
+          <distortion_t2>0.0</distortion_t2>
+          <pointCloudCutoff>0.4</pointCloudCutoff>
+        </plugin>
+      </sensor>
+    </gazebo>
   </xacro:macro>
 </robot>
